File: cyrf69103-BoB/cyrf69103-bob.brd (EAGLE design)
At the start: 18.4 x 30.7 mm, 32 parts

Commit message: Added revision and author
Other:
- board text added: "CYRF69103-BoB v0.1"
- board text added: "J Moreland Engineering LLC 22 Apr 2013"
- board text removed: "CYRF6936-BoB v0.1"
- board text removed: "J Moreland Engineering LLC 18 Apr 2013"
Changed lines of the file:
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@@
 <layer number="50" name="dxf" color="7" fill="1" visible="no" active="no"/>
 <layer number="51" name="tDocu" color="6" fill="1" visible="yes" active="yes"/>
-<layer number="52" name="bDocu" color="7" fill="1" visible="no" active="yes"/>
+<layer number="52" name="bDocu" color="7" fill="1" visible="yes" active="yes"/>
 <layer number="53" name="tPadExt" color="7" fill="1" visible="no" active="no"/>
 <layer number="54" name="bPadExt" color="1" fill="1" visible="no" active="no"/>
@@
 <wire x1="22.733" y1="28.956" x2="26.924" y2="28.956" width="0.2032" layer="51"/>
 <rectangle x1="21.082" y1="29.083" x2="23.876" y2="30.734" layer="42"/>
-<text x="25.9334" y="16.4592" size="0.889" layer="51" font="vector" ratio="15" rot="R90" align="bottom-center">CYRF6936-BoB v0.1</text>
+<text x="25.9334" y="16.4592" size="0.889" layer="51" font="vector" ratio="15" rot="R90" align="bottom-center">CYRF69103-BoB v0.1</text>
 <text x="12.827" y="16.8656" size="0.762" layer="52" font="vector" ratio="15" rot="MR270" align="bottom-center">J Moreland Engineering LLC
-18 Apr 2013</text>
+22 Apr 2013</text>
 <dimension x1="27.305" y1="38.1" x2="8.89" y2="38.1" x3="18.0975" y3="40.0304" textsize="0.8128" textratio="15" layer="47"/>
 <dimension x1="27.305" y1="7.366" x2="27.305" y2="38.1" x3="36.068" y3="22.733" textsize="0.762" textratio="15" layer="47"/>

Commit message: Screwed up that last commit.  this update include changes to the production gerber folders.  Adds hackvana to the cyrf6936-BoB and cleans up the fab notes a bit.  Still need to standardize and parameterize the creation of the gerbers.
Parts:
- R1, R2: value (none) -> 330
Changed lines of the file:
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@@
 <attribute name="VALUE" x="13.208" y="24.638" size="1.27" layer="27"/>
 </element>
-<element name="U$1" library="JCM" package="QFN40" value="CYRF69103" x="17.4752" y="20.574" rot="R90"/>
+<element name="U$1" library="JCM" package="QFN40" value="CYRF69103" x="17.4752" y="20.574" rot="R90">
+<attribute name="PARTNO" value="CYRF69103-40LFXC" x="17.4752" y="20.574" size="1.778" layer="27" rot="R90" display="off"/>
+</element>
 <element name="C2" library="SparkFun-Passives" package="0402-CAP" value="0.47uF" x="19.6088" y="14.097" rot="R270">
 <attribute name="VOLT" value="6.3" x="19.6088" y="14.097" size="1.778" layer="27" font="vector" ratio="15" rot="R270" display="off"/>
@@
 <element name="D2" library="SparkFun-LED" package="LED-0603" value="GREEN" x="13.5636" y="11.1506">
 <attribute name="PROD_ID" value="DIO-00821" x="13.5636" y="11.1506" size="1.778" layer="27" font="vector" ratio="15" display="off"/>
+<attribute name="PARTNO" value="LTST-C190KGKT" x="13.5636" y="11.1506" size="1.778" layer="27" display="off"/>
 </element>
 <element name="D1" library="SparkFun-LED" package="LED-0603" value="RED" x="13.589" y="14.097">
 <attribute name="PROD_ID" value="DIO-00819" x="13.589" y="14.097" size="1.778" layer="27" font="vector" ratio="15" display="off"/>
+<attribute name="PARTNO" value="LTST-C191TBKT" x="13.589" y="14.097" size="1.778" layer="27" display="off"/>
 </element>
-<element name="R1" library="SparkFun-Passives" package="0402-RES" value="" x="14.986" y="14.097" rot="R270"/>
-<element name="R2" library="SparkFun-Passives" package="0402-RES" value="" x="14.9352" y="11.2014" rot="R270"/>
+<element name="R1" library="SparkFun-Passives" package="0402-RES" value="330" x="14.986" y="14.097" rot="R270">
+<attribute name="PARTNO" value="CRCW0402330RJNED" x="14.986" y="14.097" size="1.778" layer="27" rot="R270" display="off"/>
+</element>
+<element name="R2" library="SparkFun-Passives" package="0402-RES" value="330" x="14.9352" y="11.2014" rot="R270">
+<attribute name="PARTNO" value="CRCW0402330RJNED" x="14.9352" y="11.2014" size="1.778" layer="27" rot="R270" display="off"/>
+</element>
 </elements>
 <signals>
